File: main board/teensyShield_progLED.kicad_pcb (KiCad board)
At the start: 2 copper layers, 34 parts, among them J1 CONN_01X14, J10 CONN_01X04, J2 CONN_01X05, J3 CONN_01X14, J4 CONN_01X03, J6 CONN_01X02, J7 CONN_01X03, J8 CONN_01X03, J9 CONN_01X03, Q1 Q_NMOS_GSD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

Commit message: Add files via upload
Parts:
- added C11: DNS, Capacitors_SMD:C_0805_HandSoldering, F.Cu at (114.8, 34.1)
- added C12: DNS, Capacitors_SMD:C_0805_HandSoldering, F.Cu at (111.8, 34.1)
- added C13: DNS, Capacitors_SMD:C_0805_HandSoldering, F.Cu at (108.8, 34.1)
- added D4: LED, Capacitors_SMD:C_0805_HandSoldering, F.Cu at (215.8, 126.1)
- added D5: LED, Capacitors_SMD:C_0805_HandSoldering, F.Cu at (150.8, 65.1)
- added J14: CONN_01X05, Pin_Headers:Pin_Header_Straight_1x05, F.Cu at (132.8, 25.1)
- added J15: CONN_01X02, Pin_Headers:Pin_Header_Straight_1x02, F.Cu at (168.8, 90.1)
- added J16: CONN_01X06, Pin_Headers:Pin_Header_Straight_1x06, F.Cu at (117.8, 25.1)
- added J5: BARREL_JACK, KicadLocalLibs:PJ-050AH, F.Cu at (110.8, 131.1)
- added PS1: PS_BUCK_MODULE, KicadLocalLibs:TC43200, F.Cu at (99.8, 122.1)
- added R10: R, Resistors_SMD:R_0805_HandSoldering, F.Cu at (197.8, 115.1)
- added R11: R, Resistors_SMD:R_0805_HandSoldering, F.Cu at (196.8, 106.1)
- added R12: 1MEG, Resistors_SMD:R_0805_HandSoldering, F.Cu at (205.8, 102.1)
- added R13: DNS, Resistors_SMD:R_0805_HandSoldering, F.Cu at (171.8, 53.1)
- added R14: 1MEG, Resistors_SMD:R_0805_HandSoldering, F.Cu at (223.8, 115.1)
- added R15: R, Resistors_SMD:R_0805_HandSoldering, F.Cu at (224.8, 123.1)
- added R16: 0, Resistors_SMD:R_0805_HandSoldering, F.Cu at (109.8, 47.1)
- added R17: R, Resistors_SMD:R_0805_HandSoldering, F.Cu at (216.8, 133.1)
- added R18: DNS, Resistors_SMD:R_0805_HandSoldering, F.Cu at (150.8, 71.1)
- added R19: 0, Resistors_SMD:R_0805_HandSoldering, F.Cu at (112.8, 47.1)
- added R20: 0, Resistors_SMD:R_0805_HandSoldering, F.Cu at (115.8, 47.1)
- added R8: R, Resistors_SMD:R_0805_HandSoldering, F.Cu at (130.8, 72.1)
- added R9: DNS, Resistors_SMD:R_0805_HandSoldering, F.Cu at (171.8, 59.1)
- added U3: MAX4373TEUA+TG071, Housings_SOIC:SOIC-8_3.9x4.9mm_Pitch1.27mm, F.Cu at (169.8, 45.1)
- added W1: TEST_1P, Mounting_Holes:MountingHole_3.2mm_M3, F.Cu at (100.0, 140.0)
- added W2: TEST_1P, Mounting_Holes:MountingHole_3.2mm_M3, F.Cu at (170.0, 140.0)
- added W3: TEST_1P, Mounting_Holes:MountingHole_3.2mm_M3, F.Cu at (100.0, 18.1)
- added W4: TEST_1P, Mounting_Holes:MountingHole_3.2mm_M3, F.Cu at (205.8, 19.1)
- added W5: TEST_1P, Mounting_Holes:MountingHole_3.2mm_M3, F.Cu at (158.8, 115.1)
- added W6: TEST_1P, Mounting_Holes:MountingHole_3.2mm_M3, F.Cu at (157.8, 80.1)
- added W7: TEST_1P, Mounting_Holes:MountingHole_3.2mm_M3, F.Cu at (106.8, 78.1)
- added W8: TEST_1P, Mounting_Holes:MountingHole_3.2mm_M3, F.Cu at (105.8, 111.1)
- D1: footprint Diodes_SMD:SMB_Handsoldering -> Diodes_SMD:DO-214AB_Handsoldering
- D2: footprint TO_SOT_Packages_SMD:SOT-23 -> Diodes_SMD:DO-214AB_Handsoldering
- D3: footprint TO_SOT_Packages_SMD:SOT-23 -> KicadLocalLibs:SOT-23_DIODE_Handsoldering
- J10: value CONN_01X04 -> CONN_01X02; footprint Pin_Headers:Pin_Header_Straight_1x04 -> Pin_Headers:Pin_Header_Straight_1x02
- J6: value CONN_01X02 -> CONN_01X04; footprint Pin_Headers:Pin_Header_Straight_1x02 -> Pin_Headers:Pin_Header_Straight_1x04
- R4: value R -> 10k
- R6: value R -> 100
- SW1: footprint Resistors_SMD:R_0805_HandSoldering -> KicadLocalLibs:R1966ABLKBLKFR
- U2: footprint TO_SOT_Packages_SMD:SOT-23 -> TO_SOT_Packages_SMD:SOT-23_Handsoldering
- moved J4 133.7 mm to (139.8, 25.1), turned to 90 degrees
- moved J9 98.4 mm to (177.8, 29.1), turned to 90 degrees
- moved J8 88.2 mm to (159.8, 25.1), turned to 90 degrees
- moved C2 84.3 mm to (192.3, 38.1), turned to 90 degrees
- moved J7 82.0 mm to (149.8, 25.1), turned to 90 degrees
- moved C6 79.6 mm to (159.8, 37.1), turned to 180 degrees
- moved C7 79.4 mm to (169.8, 132.1), turned to 270 degrees
- moved R6 77.4 mm to (168.8, 53.1), turned to 270 degrees
- moved C8 77.0 mm to (169.8, 127.1), turned to 90 degrees
- moved Q1 76.8 mm to (162.8, 45.1), turned to 90 degrees
- moved R4 74.6 mm to (168.8, 59.1), turned to 270 degrees
- moved C9 74.2 mm to (160.8, 136.1)
- moved C4 73.9 mm to (163.8, 51.6)
- moved Q2 70.6 mm to (163.8, 58.1), turned to 90 degrees
- moved C10 69.3 mm to (166.8, 68.1), turned to 180 degrees
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Connections:
- net Net-(C4-Pad1) renamed /5V_LSW
- net Net-(C4-Pad2) renamed /Q2G
- net Net-(Q1-Pad3) renamed /Q2GR
- J1 pad 2: /P0 -> /P0_RX1
- J1 pad 3: /P1 -> /P1_TX1
- J2 pad 2: /3V3 -> +3V3
- J3 pad 10: /P22 -> /P22_PWM_G
- J3 pad 11: /P23 -> /P23_PWM_R
- J3 pad 12: /3V3 -> +3V3
- J3 pad 2: /P14 -> /P14_A0
- J3 pad 8: /P20 -> /P20_PWM
- J3 pad 9: /P21 -> /P21_PWM_B
- J6 pad 1: /24V_IN -> GND
- J6 pad 2: GND -> /24V_IN
- Q1 pad 1: /P12 -> /P10
- R5 pad 2: /P12 -> /P10
Routing:
- net /24V_IN_SW_RVP: track 0.00 -> 121.3 mm
- net /24V_IN: track 0.00 -> 86.7 mm
- net /P11_MOSI: track 0.00 -> 46.2 mm
- net +5V: track 0.00 -> 41.3 mm
- net /24V_IN_SWITCHED: track 0.00 -> 36.2 mm
- net /5V_LSW: track 0.00 -> 23.4 mm
- net +3V3: track 0.00 -> 8.67 mm
- net /3V3REG: track 0.00 -> 8.29 mm
- net GND: track 0.00 -> 5.86 mm, vias 0 -> 3
- net /3V3LEDR: track 0.00 -> 3.40 mm
Other:
- net class Default: trace_width 0.25 -> 2; via_dia 0.6 -> 0.8
- rule via_min_drill: 0.3 -> 0.4
- rule via_min_size: 0.4 -> 0.8
