File: main board/teensyShield_progLED.kicad_pcb (KiCad board)
At the start: 2 copper layers, 110 x 80 mm, 84 parts, among them J1 CONN_01X14, J10 CONN_01X02, J11 CONN_01X12, J12 CONN_01X02, J13 CONN_01X02, J14 CONN_01X02, J15 CONN_01X02, J16 CONN_01X06, J17 CONN_01X02, J18 CONN_01X02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

Commit message: Moving main%20board to main\ board.
Parts:
- removed R11, R15, R7: R, Resistors_SMD:R_0805_HandSoldering
- removed R13, R9: DNS, Resistors_SMD:R_0805_HandSoldering
- removed U3: MAX4373TEUA+TG071, Housings_SOIC:SOIC-8_3.9x4.9mm_Pitch1.27mm
- added J24: CONN_02X04, Pin_Headers:Pin_Header_Straight_2x04, F.Cu at (122.0, 137.0)
- added J25: CONN_02X04, Pin_Headers:Pin_Header_Straight_2x04, F.Cu at (122.0, 125.0)
- added J26: CONN_01X03, Pin_Headers:Pin_Header_Straight_1x03, F.Cu at (125.0, 104.0)
- added J27: CONN_01X02, Pin_Headers:Pin_Header_Straight_1x02, F.Cu at (71.0, 115.0)
- added J28: CONN_01X02, Pin_Headers:Pin_Header_Straight_1x02, F.Cu at (71.0, 107.0)
- added J29: CONN_01X02, Pin_Headers:Pin_Header_Straight_1x02, F.Cu at (73.7, 138.4)
- added J30: CONN_01X02, Pin_Headers:Pin_Header_Straight_1x02, F.Cu at (71.1, 138.4)
- C4: value 1u, 0805 -> DNS
- D4: value LED -> BLUE
- D5: value LED -> GRN
- R10, R17: value R -> 220
- R12, R14: value 1MEG -> 10k
- R2: value DNS -> 0
- R23, R24, R25: value 220 -> 10
- R3, R5, R8: value R -> DNS
- moved R10 51.0 mm to (120.0, 105.0), turned to 90 degrees
- moved W6 8.91 mm to (91.5, 116.5)
- moved W7 8.72 mm to (33.0, 116.5)
- moved R17 5.38 mm to (90.0, 109.0)
- moved D4 5.32 mm to (87.0, 109.0)
- moved J5 4.40 mm to (80.0, 147.8)
- moved C1 3.80 mm to (34.2, 110.0)
- moved PS1 3.40 mm to (30.0, 106.2)
- moved W5 3.38 mm to (91.5, 144.0)
- moved W8 1.90 mm to (33.0, 144.0)
- moved C4 0.25 mm to (59.9, 121.5)
Connections:
- net /D1_5V renamed /LED3_5V
- net /D2_5V renamed /LED5_5V
- net /D3_5V renamed /LED8_5V
- net /D4_5V renamed /LED4_5V
- net /P3 renamed /P3_NOPWM
- net /P4 renamed /P4_NC
- C11 pad 1: +5VP -> +5V
- J1 pad 10: /P8 -> /P8_LED4
- J1 pad 4: /P2_P23 -> /P2_LED1
- J1 pad 7: /P5 -> /P5_LED8
- J1 pad 8: /P6 -> /P6_LED5
- J1 pad 9: /P7 -> /P7_LED3
- J20 pad 1: /LED_DOUT3 -> +5VP
- J20 pad 2: +5VP -> /LED_DOUT3
- J21 pad 1: /LED_DOUT4 -> +5VP
- J21 pad 2: +5VP -> /LED_DOUT4
- J3 pad 1: /P13_LED -> /P13_SCK
- J3 pad 2: /P14_SCK -> /P14
- J3 pad 3: /P15_A1 -> /P15_RES
- J3 pad 4: /P16 -> /P15_RES
- J3 pad 8: /P20_A6 -> /P20_LED6
- J3 pad 9: /P21 -> /P21_LED7
- J4 pad 1: /LED_DOUT1 -> +5VP
- J4 pad 2: +5VP -> /LED_DOUT1
- J6 pad 2: /24V_IN -> /24V_IN_J
- J6 pad 3: /24V_IN -> /24V_IN_J
- J8 pad 1: /LED_DOUT2 -> +5VP
- J8 pad 2: +5VP -> /LED_DOUT2
- R10 pad 1: /CIN1 -> /LED_DOUT5
- R10 pad 2: /COUT1 -> /LED1_5V_STEM
- R3 pad 2: +5VP -> +5V
- SW1 pad 2: /24V_IN -> /24V_IN_J
- U1 pad 10: GND -> /P2_LED1
- U1 pad 14: Net-(U1-Pad14) -> /LED1_5V_STEM
- U1 pad 5: /P14_SCK -> /P13_SCK
- U1 pad 6: /P12 -> /LED4_3V3
- U1 pad 7: /P9 -> /LED8_3V3
- U1 pad 8: /P8 -> /LED5_3V3
- U1 pad 9: /P7 -> /LED3_3V3
Routing:
- net GND: track 624.0 -> 233.4 mm, vias 117 -> 54
- net +5VP: track 343.8 -> 154.0 mm, vias 8 -> 0
- net (no net): track 0.00 -> 130.5 mm, vias 0 -> 16
- net /P2_P23: track 72.8 -> 0.00 mm
- net +3V3: track 167.9 -> 103.2 mm, vias 4 -> 2
- net /P0_RX1: track 62.0 -> 0.00 mm
- net /P1_TX1: track 59.8 -> 0.00 mm
- net /P2_LED1: track 0.00 -> 56.1 mm
- net /P18: track 53.1 -> 2.90 mm, vias 2 -> 0
- net /24V_IN_J: track 0.00 -> 48.7 mm
- net /LED8_3V3: track 0.00 -> 43.5 mm
- net /LED5_3V3: track 0.00 -> 40.5 mm
- net /24V_IN_SW_RVP: track 139.1 -> 100.4 mm
- net /LED3_3V3: track 0.00 -> 36.0 mm
- net /24V_IN: track 50.8 -> 15.7 mm
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Other:
- board text added: "8/8/16"
- board text added: "Rev B"
- board text added: "V D G"
- board text removed: "6/21/16"
- board text removed: "Rev A"
